File: AXIOM_connector.sch (KiCad schematic (older format))
At the start: 11 parts, among them U1001 BR24G04NUX

Commit message: fix moved plane bug, add init, done and power enable signals and optimize design
Connections:
- net ~INIT: now reaches AXIOM_SOUTH1001.B10 (IO6)
- net PWREN10: now reaches AXIOM_SOUTH1001.B11 (IO7)
- net PWREN18: now reaches AXIOM_SOUTH1001.B5 (IO1)
- net PWREN135: now reaches AXIOM_SOUTH1001.B6 (IO2)
- net DONE: now reaches AXIOM_SOUTH1001.B9 (IO5)
- no-connect marks 15 -> 10
Changed lines of the file:
@@
 S_LVDS_VCCIO
 NoConn ~ 7700 3000
-NoConn ~ 7700 3300
-NoConn ~ 7700 3400
-NoConn ~ 7700 3500
-NoConn ~ 7700 3600
-NoConn ~ 7700 3700
-NoConn ~ 7700 3800
-NoConn ~ 7700 3900
-NoConn ~ 7700 4000
 Text Notes 8450 2700 0    50   ~ 0
 swapped
@@
 Wire Wire Line
 	2900 4900 3400 4900
+Text HLabel 7800 3300 2    50   Output ~ 0
+PWREN10
+Text HLabel 7800 3400 2    50   Output ~ 0
+~INIT
+Text HLabel 7800 3800 2    50   Output ~ 0
+PWREN135
+Text HLabel 7800 3900 2    50   Output ~ 0
+PWREN18
+Text HLabel 7800 3500 2    50   Input ~ 0
+DONE
+Wire Wire Line
+	7700 3300 7800 3300
+Wire Wire Line
+	7800 3400 7700 3400
+Wire Wire Line
+	7800 3500 7700 3500
+Wire Wire Line
+	7800 3800 7700 3800
+Wire Wire Line
+	7700 3900 7800 3900
+NoConn ~ 7700 4000
+NoConn ~ 7700 3600
+NoConn ~ 7700 3700
 $EndSCHEMATC
